File: pcb/GT40.kicad_pcb (KiCad board)
At the start: 2 copper layers, 304.4 x 98.8 mm, 128 parts, among them J1 Conn_01x02, SW1 SW_PUSH, SW10 SW_PUSH, SW11 SW_PUSH, SW12 SW_PUSH, SW13 SW_PUSH, SW14 SW_PUSH, SW15 SW_PUSH, SW16 SW_PUSH, SW17 SW_PUSH, SW18 SW_PUSH, SW19 SW_PUSH, SW2 SW_PUSH, SW20 SW_PUSH, SW21 SW_PUSH, SW22 SW_PUSH, SW23 SW_PUSH, SW24 SW_PUSH, SW25 SW_PUSH, SW26 SW_PUSH, SW27 SW_PUSH, SW28 RotaryEncoder_Switch, SW29 SW_PUSH, SW3 SW_PUSH, SW30 SW_PUSH, SW31 SW_PUSH, SW32 SW_PUSH, SW33 SW_PUSH, SW34 SW_PUSH, SW35 SW_PUSH, SW36 SW_PUSH, SW37 SW_PUSH, SW38 SW_PUSH, SW39 SW_PUSH, SW4 RotaryEncoder_Switch, SW40 SW_PUSH, SW41 SW_PUSH, SW42 SW_PUSH, SW43 SW_PUSH, SW44 SW_PUSH, SW45 SW_PUSH, SW46 SW_PUSH, SW47 RotaryEncoder_Switch, SW48 SW_PUSH, SW5 SW_PUSH, SW6 SW_PUSH, SW7 SW_PUSH, SW8 SW_PUSH, SW9 SW_PUSH, U1 BLEMicroPro

Commit message: update readme.md
Parts:
- added A: LOGO, LOGO, B.Cu at (107.4, 25.3)
- added C: LOGO, LOGO, B.Cu at (171.5, 82.8)
- added D: LOGO, LOGO, B.Cu at (52.0, 102.0)
- moved SW48 41.0 mm to (149.5, 32.5)
- renumbered G** to B
Routing:
- net Reset: track 46.3 -> 14.3 mm, vias 2 -> 0
- net GND: track 894.1 -> 873.1 mm, vias 9 -> 8
- net Net-(D31-Pad1): track 24.3 -> 22.0 mm
- net Net-(L16-Pad1): track 16.6 -> 17.5 mm
